File: upsat-comms-hardware.kicad_pcb (KiCad board)
At the start: 4 copper layers, 92.5 x 92.5 mm, 314 parts, among them U1 TXCO_TG_5021CG, U10 CC1120, U12 ADT7420, U14 OPA320, U16 RF5110G, U18 FA_128_, U2 TPS79930, U3 FA_128_, U4 CC1120, U5 STM32F407VG, U6 TXCO_TG_5021CG, U8 TPS79930, Y1 Crystal, Y2 Crystal

Commit message: Edit OPA R53 resistor
It should be 180 Ohms to feed P.A AGC with 2.75 Volts.
Parts:
- R53: value 100 -> 180 Ohm
Changed lines of the file:
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@@
       (effects (font (size 1 1) (thickness 0.17)))
     )
-    (fp_text value 100 (at 0.61 1.18) (layer F.SilkS) hide
+    (fp_text value "180 Ohm" (at 0.61 1.18) (layer F.SilkS) hide
       (effects (font (size 0.5 0.5) (thickness 0.1)))
     )

Commit message: Add CC1120 bead part number
Parts:
- L1, L11: value L_Bead 0402 -> BLM15HG102SN1D
Changed lines of the file:
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@@
       (effects (font (size 1 1) (thickness 0.17)))
     )
-    (fp_text value "L_Bead 0402" (at 3.9 0 90) (layer F.SilkS) hide
+    (fp_text value BLM15HG102SN1D (at 3.9 0 90) (layer F.SilkS) hide
       (effects (font (size 1 1) (thickness 0.17)))
     )
@@
       (effects (font (size 1 1) (thickness 0.17)))
     )
-    (fp_text value "L_Bead 0402" (at 3.9 0) (layer F.SilkS) hide
+    (fp_text value BLM15HG102SN1D (at 3.9 0) (layer F.SilkS) hide
       (effects (font (size 1 1) (thickness 0.17)))
     )

Commit message: Add values for P.A RF Out matching network
Parts:
- C159: value TBD -> 6.8 pF
- C164: value 2pF -> 4 pF
- L33: value 2.7 nH -> 4.3 nH
Changed lines of the file:
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@@
       (effects (font (size 1 1) (thickness 0.17)))
     )
-    (fp_text value "2.7 nH" (at 0.61 1.18 180) (layer F.SilkS) hide
+    (fp_text value "4.3 nH" (at 0.61 1.18 180) (layer F.SilkS) hide
       (effects (font (size 0.5 0.5) (thickness 0.1)))
     )
@@
       (effects (font (size 1 1) (thickness 0.17)))
     )
-    (fp_text value 2pF (at 0.61 1.18 90) (layer F.SilkS) hide
+    (fp_text value "4 pF" (at 0.61 1.18 90) (layer F.SilkS) hide
       (effects (font (size 0.5 0.5) (thickness 0.1)))
     )
@@
       (effects (font (size 1 1) (thickness 0.17)))
     )
-    (fp_text value TBD (at 0.61 1.18 270) (layer F.SilkS) hide
+    (fp_text value "6.8 pF" (at 0.61 1.18 270) (layer F.SilkS) hide
       (effects (font (size 0.5 0.5) (thickness 0.1)))
     )
